File: RX-DATEX.kicad_pcb (KiCad board)
At the start: 4 copper layers, 65 x 100 mm, 94 parts, among them J1 Conn_01x02, J2 Conn_01x04, J3 Conn_01x03, J4 Conn_01x03, U1 Orange PI Zero 3, U10 ADuM1402xRW, U2 F0505XT-2WR2_C22388263, U3 SIM7670G-LNGV, U4 MIC29302AWU, U5 RT9193-18GB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

Commit message: update
Parts:
- C21, C24: footprint Capacitor_SMD:C_0603_1608Metric -> Capacitor_SMD:C_0805_2012Metric
- L1: value 30R/1.8A -> 47nH
- R1: value NC -> 0R
- moved C21 0.78 mm to (94.8, 106.2)
- moved C24 0.32 mm to (94.8, 108.2)
Routing:
- net GND: track 240.4 -> 217.5 mm
- net VBAT: track 91.9 -> 92.7 mm
Other:
- board text added: "+3.3V"
- board text added: "+5V"
- board text added: "A"
- board text added: "B"
- board text added: "G"
- board text added: "GND"
- board text added: "SCL"
- board text added: "SDA"
