File: SIM_Scematic.kicad_sch (KiCad schematic)
At the start: 58 parts, among them U3 SIM7670G-LNGV, U4 MIC29302AWU, U5 RT9193-18GB, U6 RT9193-33GB, U7 SMF05C_C2995323

Commit message: update
Parts:
- C21, C24: footprint Capacitor_SMD:C_0603_1608Metric -> Capacitor_SMD:C_0805_2012Metric
- L1: value 30R/1.8A -> 47nH
- R1: value NC -> 0R
Other:
- moved on the sheet: C10, C11, C12, C13, C14, C15, C16, C17, C18, C19, C20, C21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
