File: RX-PSU-AC.kicad_pcb (KiCad board)
At the start: 2 copper layers, 65 x 50 mm, 21 parts, among them J1 Conn_01x02, J2 Conn_01x04, J3 Conn_01x02, Q1 BSS138, Q2 BSS138, U1 HLK-10M05, U2 INA219AxD, U3 MCP1825S

Commit message: update
Parts:
- added TP1: TestPoint, TestPoint:TestPoint_Pad_D1.0mm, B.Cu at (112.0, 61.0)
- added TP2: TestPoint, TestPoint:TestPoint_Pad_D1.0mm, B.Cu at (112.0, 64.0)
- U3: value MCP1825S -> ME6211C33M5; footprint Package_TO_SOT_SMD:SOT-223-3_TabPin2 -> Package_TO_SOT_SMD:SOT-23-5
- moved C2 9.66 mm to (109.0, 61.0), turned to 0 degrees
- moved U3 2.50 mm to (109.0, 65.5), turned to -90 degrees
- moved C3 1.50 mm to (109.0, 70.0)
Connections:
- U3 pad 3: +3V3 -> +5V
Routing:
- net +5V: track 51.7 -> 72.9 mm
- net GND: track 53.1 -> 47.5 mm, vias 120 -> 143
- net +3V3: track 43.3 -> 46.2 mm
