File: RX-PSU-AC.kicad_sch (KiCad schematic)
At the start: 20 parts, among them J1 Conn_01x02, J2 Conn_01x04, J3 Conn_01x02, Q1 BSS138, Q2 BSS138, U1 HLK-10M05, U2 INA219AxD, U3 MCP1825S

Commit message: update
Parts:
- removed U3: MCP1825S, Package_TO_SOT_SMD:SOT-223-3_TabPin2, symbol Regulator_Linear:MCP1825S
- added TP1, TP2: TestPoint, TestPoint:TestPoint_Pad_D1.0mm, symbol Connector:TestPoint
- added U3: ME6211C33M5, Package_TO_SOT_SMD:SOT-23-5, symbol Regulator_Linear:ME6211C33M5
Connections:
- net +3V3: now also TP2.1, U3.5 (V_{OUT})
- net +5V: now also TP1.1, U3.1 (V_{IN}), U3.3 (CE)
- net GND: now also U3.2 (V_{SS})
Other:
- moved on the sheet: C2, C3, J2
